Commit message: feat: add RL walk policy deployment and DART physics support
- Add walk_controller.py for deploying trained RL policy (model_1700.pt)
- Add gazebo_walk.launch with DART physics engine
- Update URDF: add transmissions, friction, effort limits (100 Nm)
- Update stand_controller.py to only control Go2 joints
- Add empty_world_custom.world with DART physics config

Co-Authored-By: Claude Opus 4.6 (1M context) <noreply@anthropic.com>

File: src/leg_manipulator/urdf/go2_with_diy_leg.urdf (robot description, URDF)
Before this commit: robot go2_with_diy_leg, 42 links, 41 joints
Links:
- link RL_calflower: mass 0.001 -> None
- link RL_calflower1: mass 0.001 -> None
- link RR_calflower: mass 0.001 -> None
- link RR_calflower1: mass 0.001 -> None
- link front_camera: mass 0.001 -> None
- link imu: mass 0.001 -> 0
- link radar: mass 0.001 -> 0
Joints:
- joint FL_calf_joint: limit lower=-2.9 upper=-1.2 effort=45.43 velocity=15.70 -> lower=-2.9 upper=-1.2 effort=100.0 velocity=15.70
- joint FL_diy_joint1: limit lower=0 upper=0.1 effort=40 velocity=0.01 -> lower=0 upper=0.1 effort=100 velocity=1
- joint FL_diy_joint2: limit lower=-2.4 upper=0.67 effort=4.9 velocity=7.85 -> lower=-2.4 upper=0.67 effort=100 velocity=1
- joint FL_diy_joint3: limit lower=-1.42 upper=1.45 effort=1.39 velocity=10.47 -> lower=-1.42 upper=1.45 effort=100 velocity=1
- joint FL_diy_joint4: limit lower=-0.17 upper=1.4 effort=1.39 velocity=10.47 -> lower=-0.17 upper=1.4 effort=100 velocity=1
- joint FL_hip_joint: limit lower=-1.0472 upper=1.0472 effort=23.7 velocity=30.1 -> lower=-1.0472 upper=1.0472 effort=100.0 velocity=30.1
- joint FL_thigh_joint: limit lower=-1.5708 upper=3.4907 effort=23.7 velocity=30.1 -> lower=-1.5708 upper=3.4907 effort=100.0 velocity=30.1
- joint FR_calf_joint: limit lower=-2.9 upper=-1.2 effort=45.43 velocity=15.70 -> lower=-2.9 upper=-1.2 effort=100.0 velocity=15.70
- joint FR_hip_joint: limit lower=-1.0472 upper=1.0472 effort=23.7 velocity=30.1 -> lower=-1.0472 upper=1.0472 effort=100.0 velocity=30.1
- joint FR_thigh_joint: limit lower=-1.5708 upper=3.4907 effort=23.7 velocity=30.1 -> lower=-1.5708 upper=3.4907 effort=100.0 velocity=30.1
- joint RL_calf_joint: limit lower=-2.7227 upper=-0.83776 effort=45.43 velocity=15.70 -> lower=-2.7227 upper=-0.83776 effort=100.0 velocity=15.70
- joint RL_hip_joint: limit lower=-1.0472 upper=1.0472 effort=23.7 velocity=30.1 -> lower=-1.0472 upper=1.0472 effort=100.0 velocity=30.1
- joint RL_thigh_joint: limit lower=-0.5236 upper=4.5379 effort=23.7 velocity=30.1 -> lower=-0.5236 upper=4.5379 effort=100.0 velocity=30.1
- joint RR_calf_joint: limit lower=-2.7227 upper=-0.83776 effort=45.43 velocity=15.70 -> lower=-2.7227 upper=-0.83776 effort=100.0 velocity=15.70
- joint RR_hip_joint: limit lower=-1.0472 upper=1.0472 effort=23.7 velocity=30.1 -> lower=-1.0472 upper=1.0472 effort=100.0 velocity=30.1
- joint RR_thigh_joint: limit lower=-0.5236 upper=4.5379 effort=23.7 velocity=30.1 -> lower=-0.5236 upper=4.5379 effort=100.0 velocity=30.1
- joint diy_joint1: limit lower=0 upper=0.1 effort=40 velocity=0.01 -> lower=0 upper=0.1 effort=100 velocity=1
- joint diy_joint2: limit lower=-2.4 upper=0.67 effort=4.9 velocity=7.85 -> lower=-2.4 upper=0.67 effort=100 velocity=1
- joint diy_joint3: limit lower=-1.42 upper=1.45 effort=1.39 velocity=10.47 -> lower=-1.42 upper=1.45 effort=100 velocity=1
- joint diy_joint4: limit lower=-0.17 upper=1.4 effort=1.39 velocity=10.47 -> lower=-0.17 upper=1.4 effort=100 velocity=1
