Commit message: fix: restructure repo, correct joint mapping, add IMU and DART support
- Move git tracking from src/leg_manipulator/ to repo root
- Fix joint order mapping: policy uses type-grouped order, URDF uses leg-grouped
- Add IMU sensor plugin to URDF for correct observations
- Fix zero-mass links (imu, radar) causing DART instability
- Add friction/contact params matching training config
- Restore original effort limits (hip/thigh=23.7, calf=45.43)
- Use DART physics engine for better contact solving
- Add walk_controller.py and pybullet_sim2sim.py

Co-Authored-By: Claude Opus 4.6 (1M context) <noreply@anthropic.com>

File: urdf/go2_with_diy_leg.urdf (robot description, URDF)
Before this commit: robot go2_with_diy_leg, 42 links, 41 joints
Links:
- link imu: mass 0 -> 0.001
- link radar: mass 0 -> 0.001
Joints:
- joint FL_calf_joint: limit lower=-2.9 upper=-1.2 effort=100.0 velocity=15.70 -> lower=-2.9 upper=-1.2 effort=45.43 velocity=15.70
- joint FL_hip_joint: limit lower=-1.0472 upper=1.0472 effort=100.0 velocity=30.1 -> lower=-1.0472 upper=1.0472 effort=23.7 velocity=30.1
- joint FL_thigh_joint: limit lower=-1.5708 upper=3.4907 effort=100.0 velocity=30.1 -> lower=-1.5708 upper=3.4907 effort=23.7 velocity=30.1
- joint FR_calf_joint: limit lower=-2.9 upper=-1.2 effort=100.0 velocity=15.70 -> lower=-2.9 upper=-1.2 effort=45.43 velocity=15.70
- joint FR_hip_joint: limit lower=-1.0472 upper=1.0472 effort=100.0 velocity=30.1 -> lower=-1.0472 upper=1.0472 effort=23.7 velocity=30.1
- joint FR_thigh_joint: limit lower=-1.5708 upper=3.4907 effort=100.0 velocity=30.1 -> lower=-1.5708 upper=3.4907 effort=23.7 velocity=30.1
- joint RL_calf_joint: limit lower=-2.7227 upper=-0.83776 effort=100.0 velocity=15.70 -> lower=-2.7227 upper=-0.83776 effort=45.43 velocity=15.70
- joint RL_hip_joint: limit lower=-1.0472 upper=1.0472 effort=100.0 velocity=30.1 -> lower=-1.0472 upper=1.0472 effort=23.7 velocity=30.1
- joint RL_thigh_joint: limit lower=-0.5236 upper=4.5379 effort=100.0 velocity=30.1 -> lower=-0.5236 upper=4.5379 effort=23.7 velocity=30.1
- joint RR_calf_joint: limit lower=-2.7227 upper=-0.83776 effort=100.0 velocity=15.70 -> lower=-2.7227 upper=-0.83776 effort=45.43 velocity=15.70
- joint RR_hip_joint: limit lower=-1.0472 upper=1.0472 effort=100.0 velocity=30.1 -> lower=-1.0472 upper=1.0472 effort=23.7 velocity=30.1
- joint RR_thigh_joint: limit lower=-0.5236 upper=4.5379 effort=100.0 velocity=30.1 -> lower=-0.5236 upper=4.5379 effort=23.7 velocity=30.1

Commit message: fix: add DIY joint position control, fix ang_vel observation, switch to DART
- Add DIY joint transmissions (PositionJointInterface) and controllers
- Fix angular velocity observation: IMU already outputs body frame, remove redundant rotation
- Restore DIY revolute effort limits (joint2=4.9, joint3/4=1.39)
- Switch physics engine to DART
- Update walk_model path

Co-Authored-By: Claude Opus 4.6 (1M context) <noreply@anthropic.com>

File: urdf/go2_with_diy_leg.urdf (robot description, URDF)
Before this commit: robot go2_with_diy_leg, 42 links, 41 joints
Joints:
- joint FL_diy_joint2: limit lower=-2.4 upper=0.67 effort=100 velocity=1 -> lower=-2.4 upper=0.67 effort=4.9 velocity=7.85
- joint FL_diy_joint3: limit lower=-1.42 upper=1.45 effort=100 velocity=1 -> lower=-1.42 upper=1.45 effort=1.39 velocity=10.47
- joint FL_diy_joint4: limit lower=-0.17 upper=1.4 effort=100 velocity=1 -> lower=-0.17 upper=1.4 effort=1.39 velocity=10.47
- joint diy_joint2: limit lower=-2.4 upper=0.67 effort=100 velocity=1 -> lower=-2.4 upper=0.67 effort=4.9 velocity=7.85
- joint diy_joint3: limit lower=-1.42 upper=1.45 effort=100 velocity=1 -> lower=-1.42 upper=1.45 effort=1.39 velocity=10.47
- joint diy_joint4: limit lower=-0.17 upper=1.4 effort=100 velocity=1 -> lower=-0.17 upper=1.4 effort=1.39 velocity=10.47
