Commit message: feat: vision-driven walk-and-grasp demo + mesh reorganization
walk_and_grasp.py: end-to-end pipeline driving the trained Go2+DIY-leg walk
policy to find a red dumbbell with the head_cam, walk up, extend the arm,
servo-align EE to the bar, close the gripper, and verify the grasp via
active arm-lift (cube must rise with the arm to count as held).

leg_manipulator/mjcf/build_mjcf.py: Python generator that builds go2_diyleg.xml
from the URDF, adds the head_cam, target platform, dumbbell target, and a
keyframe consistent with the trained policy's standing pose.

Repo cleanup:
- Move stock Go2 collada/obj meshes into leg_manipulator/go2_description/
- Move DIY-arm STLs into leg_manipulator/meshes/
- Drop the obsolete URDF→MJCF converter; build_mjcf.py replaces it
- Drop the old 1700-step ONNX; current policy is the 6200-step one
- Add .gitignore for __pycache__, recorded *.mp4, and one-off _diag_*.py

Co-Authored-By: Claude Opus 4.7 <noreply@anthropic.com>

File: leg_manipulator/urdf/go2_with_diy_leg.urdf (robot description, URDF)
Before this commit: robot go2_with_diy_leg, 42 links, 41 joints
Links:
- added link FL_diy_foot, mass 0.04; collision mesh filename=package://go2_description/dae/foot.dae scale=1.3 1.3 1.3; visual mesh filename=package://go2_description/dae/foot.dae scale=1.3 1.3 1.3
- added link FR_diy_foot, mass 0.04; collision mesh filename=package://go2_description/dae/foot.dae scale=1.3 1.3 1.3; visual mesh filename=package://go2_description/dae/foot.dae scale=1.3 1.3 1.3
- link FL_diy_base_link: mass 0.228916745240302 -> 0.209323724052629
- link FL_diy_link1: mass 0.0589546671844344 -> 0.0589546671873471
- link FL_diy_link2: mass 0.0492722298663148 -> 0.049272
- link FL_diy_link3: mass 0.111402715752738 -> 0.0862103337643177
- link FL_diy_link4: mass 0.0268787641612815 -> 0.026431100728336
- link FL_hip: geometry collision cylinder length=0.04 radius=0.046; visual mesh filename=package://go2_description/dae/hip.dae
- link FL_thigh: geometry collision box size=0.213 0.0245 0.034; visual mesh filename=package://go2_description/dae/thigh.dae
- link FR_hip: geometry collision cylinder length=0.04 radius=0.046; visual mesh filename=package://go2_description/dae/hip.dae
- link FR_thigh: geometry collision box size=0.213 0.0245 0.034; visual mesh filename=package://go2_description/dae/thigh_mirror.dae
- link RL_calf: geometry collision cylinder length=0.12 radius=0.013; visual mesh filename=package://go2_description/dae/calf.dae
- link RL_calflower: mass 0.001 -> None
- link RL_calflower1: mass 0.001 -> None
- link RL_foot: geometry collision sphere radius=0.022; visual mesh filename=package://go2_description/dae/foot.dae
- link RL_hip: geometry collision cylinder length=0.04 radius=0.046; visual mesh filename=package://go2_description/dae/hip.dae
- link RL_thigh: geometry collision box size=0.213 0.0245 0.034; visual mesh filename=package://go2_description/dae/thigh.dae
- link RR_calf: geometry collision cylinder length=0.12 radius=0.013; visual mesh filename=package://go2_description/dae/calf_mirror.dae
- link RR_calflower: mass 0.001 -> None
- link RR_calflower1: mass 0.001 -> None
- link RR_foot: geometry collision sphere radius=0.022; visual mesh filename=package://go2_description/dae/foot.dae
- link RR_hip: geometry collision cylinder length=0.04 radius=0.046; visual mesh filename=package://go2_description/dae/hip.dae
- link RR_thigh: geometry collision box size=0.213 0.0245 0.034; visual mesh filename=package://go2_description/dae/thigh_mirror.dae
- link base: geometry collision box size=0.3762 0.0935 0.114; visual mesh filename=package://go2_description/dae/base.dae
- link diy_base_link: mass 0.228916745240302 -> 0.209323724052629
- link diy_link1: mass 0.0589546671844344 -> 0.0589546671873471
- link diy_link2: mass 0.0492722298663148 -> 0.049272
- link diy_link3: mass 0.111402715752738 -> 0.0862103337643177
- link diy_link4: mass 0.0268787641612815 -> 0.026431100728336
- link front_camera: mass 0.001 -> None
- link imu: mass 0.001 -> 0
- link radar: mass 0.001 -> 0
Joints:
- added joint FL_diy_foot_joint: type fixed, parent FL_diy_base_link, child FL_diy_foot, origin xyz=0.196 -0.045 0.0 rpy=1.5708 0 3.35, axis 0 0 0
- added joint FR_diy_foot_joint: type fixed, parent diy_base_link, child FR_diy_foot, origin xyz=0.196 -0.045 0.0 rpy=1.5708 0 3.35, axis 0 0 0
- joint FL_calf_joint: axis 0 1 0 -> 0 0 1; limit lower=-2.9 upper=-1.2 effort=45.43 velocity=15.70 -> lower=0.99 upper=2.82 effort=45.43 velocity=15.70; origin xyz=0 -0.002 -0.212 rpy=0 -1.5708 0 -> xyz=0 -0.002 -0.212 rpy=1.5708 1.5708 0
- joint FL_diy_joint1: axis 1 0 0 -> -1 -0.0012292 0; limit lower=0 upper=0.1 effort=40 velocity=0.01 -> lower=0 upper=0.105 effort=100 velocity=1; origin xyz=-0.022741 -5E-05 0.032 rpy=3.1416 0 0 -> xyz=0.022502 -0.034022 0 rpy=0 0 0; type prismatic -> fixed
- joint FL_diy_joint2: axis 0 -1 0 -> 0 0 -1; limit lower=-2.4 upper=0.67 effort=4.9 velocity=7.85 -> lower=-2.2 upper=0.08 effort=100 velocity=1; origin xyz=-0.145982705510586 -0.0292000000000024 0.0227 rpy=0 0 0 -> xyz=0.14708 0.022931 -0.0291 rpy=0 0 0; type revolute -> fixed
- joint FL_diy_joint3: axis 0.46021 0 0.88781 -> -0.6572 0.75372 0; limit lower=-1.42 upper=1.45 effort=1.39 velocity=10.47 -> lower=-1.2 upper=1.2 effort=100 velocity=1; origin xyz=-0.050675 0.029 0.017145 rpy=0 0 0 -> xyz=0.045837 0.027894 0.029 rpy=0 0 0; type revolute -> fixed
- joint FL_diy_joint4: axis 0.014315 0.99987 -0.0074203 -> 0.047892 0.041759 0.99798; limit lower=-0.17 upper=1.4 effort=1.39 velocity=10.47 -> lower=0.2 upper=2.3 effort=100 velocity=1; origin xyz=-0.12194 -0.015927 0.044362 rpy=0 0 0 -> xyz=0.083867 0.052256 -0.024248 rpy=0 0 0; type revolute -> fixed
- joint FR_calf_joint: axis 0 1 0 -> 0 0 1; limit lower=-2.9 upper=-1.2 effort=45.43 velocity=15.70 -> lower=0.99 upper=2.82 effort=45.43 velocity=15.70; origin xyz=0 0.002 -0.212 rpy=0 -1.5708 0 -> xyz=0 0.002 -0.212 rpy=1.5708 1.5708 0
- joint diy_joint1: axis 1 0 0 -> -1 -0.0012292 0; limit lower=0 upper=0.1 effort=40 velocity=0.01 -> lower=0 upper=0.105 effort=100 velocity=1; origin xyz=-0.022741 -5E-05 0.032 rpy=3.1416 0 0 -> xyz=0.022502 -0.034022 0 rpy=0 0 0; type prismatic -> fixed
- joint diy_joint2: axis 0 -1 0 -> 0 0 -1; limit lower=-2.4 upper=0.67 effort=4.9 velocity=7.85 -> lower=-2.2 upper=0.08 effort=100 velocity=1; origin xyz=-0.145982705510586 -0.0292000000000024 0.0227 rpy=0 0 0 -> xyz=0.14708 0.022931 -0.0291 rpy=0 0 0; type revolute -> fixed
- joint diy_joint3: axis 0.46021 0 0.88781 -> -0.6572 0.75372 0; limit lower=-1.42 upper=1.45 effort=1.39 velocity=10.47 -> lower=-1.2 upper=1.2 effort=100 velocity=1; origin xyz=-0.050675 0.029 0.017145 rpy=0 0 0 -> xyz=0.045837 0.027894 0.029 rpy=0 0 0; type revolute -> fixed
- joint diy_joint4: axis 0.014315 0.99987 -0.0074203 -> 0.047892 0.041759 0.99798; limit lower=-0.17 upper=1.4 effort=1.39 velocity=10.47 -> lower=0.2 upper=2.3 effort=100 velocity=1; origin xyz=-0.12194 -0.015927 0.044362 rpy=0 0 0 -> xyz=0.083867 0.052256 -0.024248 rpy=0 0 0; type revolute -> fixed
